File: CPU09IDE/CPU09IDE/CPU09IDE.kicad_sch (KiCad schematic)
At the start: 48 parts, among them J1 BUS, J2 IDE, J34 Conn_02x03_Odd_Even, J5 Jumper_3_Open, J6 Interrupt, U1 74HC74, U10 74HC273, U11 74HC573, U12 74HC161, U13 74HC573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

Commit message: IDE schematic title ch.
Other:
- title: CPUXXCMI Board -> CPU09IDE Board
