File: ExorsetFloppy/Exorset_Floppy/Exorset_Floppy.kicad_pcb (KiCad board)
At the start: 2 copper layers, 160 x 100 mm, 89 parts, among them J1 BUS, J10 Conn_01x01, J11 Conn_01x01, J12 Conn_01x01, J13 Conn_01x01, J14 Conn_01x01, J15 Conn_01x01, J16 Conn_01x01, J17 Conn_01x01, J18 Conn_01x01, J19 Conn_01x01, J2 Floppy, J20 Conn_01x01, J3 Conn_01x01, J4 Conn_01x01, J5 Conn_01x01, J6 Conn_01x01, J7 Conn_01x17, J8 Conn_01x01, J9 Conn_01x01, Q1 BC337, U1 GAL22V10, U10 GAL16V8, U11 74HCT74, U12 74HCT74, U13 74LS91, U14 74HCT74, U15 74HCT04, U16 74HCT74, U17 74HCT00, U18 74HCT74, U19 74LS76, U2 74HCT74, U20 68B21, U21 MC4024, U22 74LS157, U23 74LS123, U24 74HC164, U25 74LS04, U27 MC4044, U28 74F163, U29 74F163, U3 74HC245, U34 6852_DIL24, U4 MC8506, U5 74F163, U6 27C32, U7 74LS240, U8 74LS244, U9 NE555P

Commit message: some small adjustments
Parts:
- added J21: Conn_01x01, Connector_PinHeader_1.27mm:PinHeader_1x01_P1.27mm_Vertical, F.Cu at (193.3, 124.3)
- added J22: Conn_01x01, Connector_PinHeader_1.27mm:PinHeader_1x01_P1.27mm_Vertical, F.Cu at (189.7, 124.3)
- added JP8: CLOCKSRC, Jumper:SolderJumper-3_P1.3mm_Bridged12_RoundedPad1.0x1.5mm_NumberLabels, F.Cu at (155.8, 52.8)
- added Y1: 1M, Oscillator:Oscillator_DIP-8, F.Cu at (208.0, 62.2)
- RN2: value 4k7 -> 1k
- U7: value 74LS240 -> 74HCT240
- U8: value 74LS244 -> 74HCT244
- U9: value NE555P -> NE7555P
Connections:
- U14 pad 3: /B_E -> Net-(JP8-C)
- U20 pad 7: unconnected-(U20-PA5-Pad7) -> /Floppy Logic/PA5
Routing:
- net /Floppy Logic/PA5: track 0.00 -> 91.5 mm, vias 0 -> 1
- net /Floppy Logic/~{TG43}: track 0.00 -> 69.6 mm, vias 0 -> 1
- net Net-(JP8-B): track 0.00 -> 60.8 mm
- net GND: track 937.4 -> 970.8 mm, vias 113 -> 169
- net Net-(JP8-C): track 0.00 -> 29.1 mm, vias 0 -> 1
- net +5V: track 925.2 -> 953.2 mm
- net /B_E: track 197.5 -> 210.9 mm, vias 5 -> 6
- net /Floppy Logic/RAW_DATA: track 77.7 -> 75.5 mm
- net Net-(U20-CB2): track 51.3 -> 50.0 mm
- net /Floppy Logic/PB2: track 110.2 -> 109.0 mm
- net /Floppy Logic/CLK_U5_15: track 85.3 -> 86.0 mm
- net /Floppy Logic/PB0: track 111.1 -> 111.8 mm
- net /Floppy Logic/~{WDAT}: track 71.8 -> 71.2 mm
- net /BA2: track 114.8 -> 114.2 mm
- net /Floppy Logic/STEP: track 40.5 -> 39.9 mm
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Other:
- board text added: "CLKSRC"
- board text added: "JP8 left: Clock from Bus right: Clock from Y1."
- board text added: "PA5"
- board text added: "TG43"
