File: ExorsetFloppy/Exorset_Floppy/floppyLogic.kicad_sch (KiCad schematic)
At the start: 64 parts, among them J2 Floppy, J3 Conn_01x01, J4 Conn_01x01, J5 Conn_01x01, J6 Conn_01x01, Q1 BC337, U10 GAL22V10, U11 74HCT74, U12 74HCT74, U121 74LS624, U13 74LS91, U15 74HCT04, U16 74HCT74, U17 74HCT00, U18 74HCT74, U19 74LS76, U2 74HCT74, U20 68B21, U21 MC4024, U22 74LS157, U221 74LS627, U23 74LS123, U24 74HC164, U27 MC4044, U28 74F163, U29 74F163, U34 6852_DIL24, U4 MC8506, U5 74F163, U7 74LS240, U8 74LS244, U9 NE555P

Commit message: Board finished, GALS added
Parts:
- removed D3: BAT42, Diode_THT:D_5W_P10.16mm_Horizontal, symbol Device:D_Schottky_Small_Filled
- removed J4, J5, J6: Conn_01x01, Connector_PinHeader_1.27mm:PinHeader_1x01_P1.27mm_Vertical, symbol Connector_Generic:Conn_01x01
- removed U10: GAL22V10, Package_DIP:DIP-24_W7.62mm, symbol my_ics_new:GAL22V10
- removed unit 3 of U11
- removed unit 3 of U12
- removed U121: 74LS624, Package_DIP:DIP-14_W7.62mm, symbol my_ics_new:74LS624
- removed unit 7 of U15
- removed unit 3 of U16
- removed unit 5 of U17
- removed unit 3 of U18
- removed unit 3 of U19
- removed unit 2 of U19
- removed unit 3 of U2
- removed U221: 74LS627, Package_DIP:DIP-14_W7.62mm, symbol my_ics_new:74LS627
- removed unit 3 of U23
- added D3: BAS40-04, Package_TO_SOT_SMD:SOT-23_Handsoldering, symbol Diode:BAS40-04
- added J10, J11, J12, J13, J14, J15, J16, J17, J18, J8, J9: Conn_01x01, Connector_PinHeader_1.27mm:PinHeader_1x01_P1.27mm_Vertical, symbol Connector_Generic:Conn_01x01
- added J19, J20: Conn_01x01, Connector_PinHeader_2.54mm:PinHeader_1x01_P2.54mm_Vertical, symbol Connector_Generic:Conn_01x01
- added J7: Conn_01x17, Connector_PinHeader_2.54mm:PinHeader_1x17_P2.54mm_Vertical, symbol Connector_Generic:Conn_01x17
- added U10: GAL16V8, Package_DIP:DIP-20_W7.62mm, symbol Logic_Programmable:GAL16V8
- added U25: 74LS04, Package_DIP:DIP-14_W7.62mm, symbol 74xx:74LS04
- C8, C9: footprint Capacitor_THT:CP_Radial_D10.0mm_P5.00mm -> Capacitor_THT:CP_Radial_D8.0mm_P5.00mm
- D1, D2: footprint Diode_THT:D_5W_P10.16mm_Horizontal -> Diode_SMD:D_1206_3216Metric_Pad1.42x1.75mm_HandSolder
- Q1: footprint Package_TO_SOT_THT:TO-92L -> Package_TO_SOT_THT:TO-92L_Wide
- U21: now fitted
Connections:
- net +5V: now also U10.20 (VCC)
- net CRC_DATA: now also U10.13 (IO7)
- net CRC_DOUT: now also U10.11 (I10/~{OE})
- net D: now also J14.1 (Pin_1)
- net FAST: now also U10.9 (I9)
- net F_A: now also J7.8 (Pin_8)
- net F_B: now also J7.3 (Pin_3)
- net GND: now also J19.1 (Pin_1), J20.1 (Pin_1), U10.10 (GND)
- net INUSE: now also J7.2 (Pin_2)
- net PB0: now also U25.5
- net PB2: now also U25.11
- net RAW_DATA: now also J13.1 (Pin_1)
- net RCLK: now also J15.1 (Pin_1)
- net RESET: now also U25.6, U25.9
- net RXD: now also J18.1 (Pin_1)
- net SLOW: now also U10.8 (I8)
- net TUF: now also U25.13
- net TUF#: now also U25.4
- net WRITE/~{READ}: now also U25.10
- net ~{6820_CS}: now also U10.7 (I7)
- net ~{6852_CS}: now also U10.6 (I6)
- net ~{8x_RD_CLK}: now also J16.1 (Pin_1)
- net ~{DIR}: now also J7.9 (Pin_9)
- net ~{DS0}: now also J7.5 (Pin_5)
- net ~{DS1}: now also J7.6 (Pin_6)
- net ~{DS2}: now also J7.7 (Pin_7)
- net ~{F_MODE}: now also J7.1 (Pin_1)
- net ~{F_RDY}: now also J7.17 (Pin_17)
- net ~{F_WG}: now also J7.12 (Pin_12)
- net ~{IDX}: now also J7.4 (Pin_4)
- net ~{RDAT}: now also J7.15 (Pin_15)
- net ~{RESET}: now also U25.8
- net ~{RFF}: now also D3.3, U10.19 (IO1)
- net ~{SIDE1}: now also J7.16 (Pin_16)
- net ~{STEP}: now also J7.10 (Pin_10)
- net ~{TRK00}: now also J7.13 (Pin_13)
- net ~{TUF}: now also U25.12, U25.3
- net ~{WDAT}: now also J7.11 (Pin_11)
- net ~{WPT}: now also J7.14 (Pin_14)
- net at U2.5 (Q): now also U10.1 (I1/CLK)
- net at U2.6 (~{Q}): now also U10.2 (I2)
- net at C21.1, R2.1, U9.6 (THR)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: now also D3.1
- net at U12.2 (D), U16.5 (Q): now also J17.1 (Pin_1)
- net at U8.15 (I2b): now also J8.1 (Pin_1)
- net at U8.5 (O2b): now also J9.1 (Pin_1)
- net at U18.12 (D), U18.5 (Q): now also J12.1 (Pin_1)
- net SWCLK: no longer names the net of U34.3 (RXClk), U34.4 (TXClk)
- net SWCLK: now also U25.2
- new net: J10.1 (Pin_1), U10.17 (I03)
- new net: J11.1 (Pin_1), U10.18 (IO2)
- new net BA11: U10.15 (IO5)
- new net BA12: U10.14 (IO6)
- new net BA13: U10.5 (I5)
- new net BA14: U10.4 (I4)
- new net BA15: U10.3 (I3)
- new net SEL: U10.16 (IO4)
- new net ~{SWCLK}: U10.12 (IO8), U25.1
- no-connect marks 53 -> 42
Other:
- note added: "Clock (500kHz nom.)"
- note added: "G2"
- note removed: "12v from Where? ~{F_MODE} connected? ~{SIDE} connected? 74161 can be replaced by 74163."
- note removed: "Clock"
- moved on the sheet: J2, U34

Commit message: some small adjustments
Parts:
- added J21, J22: Conn_01x01, Connector_PinHeader_1.27mm:PinHeader_1x01_P1.27mm_Vertical, symbol Connector_Generic:Conn_01x01
- RN2: value 4k7 -> 1k
- U7: value 74LS240 -> 74HCT240
- U8: value 74LS244 -> 74HCT244
- U9: value NE555P -> NE7555P
Connections:
- net ~{TG43}: now also J21.1 (Pin_1)
- net PA5: now reaches U20.7 (PA5)
- net PA5: now also J22.1 (Pin_1)
- no-connect marks 42 -> 41
Other:
- moved on the sheet: JP1
Changed lines of the file:
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@@
 	)
 	(no_connect
-		(at 54.61 35.56)
-	)
-	(no_connect
 		(at 245.11 60.96)
 	)
@@
 	(wire
 		(pts
+			(xy 71.12 40.64) (xy 78.74 40.64)
+		)
+		(stroke
+			(width 0)
+			(type default)
+		)
+	)
+	(wire
+		(pts
 			(xy 54.61 58.42) (xy 66.04 58.42)
 		)
@@
 	(wire
 		(pts
-			(xy 342.9 80.01) (xy 351.79 80.01)
+			(xy 346.71 80.01) (xy 355.6 80.01)
 		)
 		(stroke
@@
 	(wire
 		(pts
+			(xy 66.04 35.56) (xy 54.61 35.56)
+		)
+		(stroke
+			(width 0)
+			(type default)
+		)
+	)
+	(wire
+		(pts
 			(xy 271.78 142.24) (xy 278.13 142.24)
 		)
@@
 		)
 	)
+	(label "PA5"
+		(at 71.12 40.64 0)
+		(effects
+			(font
+				(size 1.27 1.27)
+			)
+			(justify left bottom)
+		)
+	)
 	(label "HLD"
 		(at 66.04 33.02 180)
@@
 	)
 	(label "~{F_MODE}"
-		(at 342.9 80.01 0)
+		(at 346.71 80.01 0)
 		(effects
 			(font
@@
 		)
 	)
+	(label "PA5"
+		(at 66.04 35.56 180)
+		(effects
+			(font
+				(size 1.27 1.27)
+			)
+			(justify right bottom)
+		)
+	)
 	(label "BA13"
 		(at 134.62 57.15 0)
@@
 	(symbol
 		(lib_id "power:+5V")
-		(at 355.6 73.66 0)
+		(at 359.41 73.66 0)
 		(unit 1)
 		(exclude_from_sim no)
@@
 		(dnp no)
 		(property "Reference" "#PWR087"
-			(at 355.6 77.47 0)
+			(at 359.41 77.47 0)
 			(effects
 				(font
@@
 		)
 		(property "Value" "+5V"
-			(at 355.6 69.596 0)
+			(at 359.41 69.596 0)
 			(effects
 				(font
@@
 		)
 		(property "Footprint" ""
-			(at 355.6 73.66 0)
+			(at 359.41 73.66 0)
 			(effects
 				(font
@@
 		)
 		(property "Datasheet" ""
-			(at 355.6 73.66 0)
+			(at 359.41 73.66 0)
 			(effects
 				(font
@@
 		)
 		(property "Description" "Power symbol creates a global label with name \"+5V\""
-			(at 355.6 73.66 0)
+			(at 359.41 73.66 0)
 			(effects
 				(font
@@
 			)
 		)
-		(property "Value" "4k7"
+		(property "Value" "1k"
 			(at 370.84 48.5139 0)
 			(effects
@@
 			)
 		)
-		(property "Value" "74LS244"
+		(property "Value" "74HCT244"
 			(at 322.1833 63.5 0)
 			(effects
@@
 		(fields_autoplaced yes)
 		(property "Reference" "U9"
-			(at 268.8941 66.04 0)
+			(at 268.8433 66.04 0)
 			(effects
 				(font
@@
 			)
 		)
-		(property "Value" "NE555P"
-			(at 268.8941 68.58 0)
+		(property "Value" "NE7555P"
+			(at 268.8433 68.58 0)
 			(effects
 				(font
@@
 	(symbol
 		(lib_id "Jumper:Jumper_3_Open")
-		(at 355.6 80.01 270)
+		(at 359.41 80.01 270)
 		(unit 1)
 		(exclude_from_sim yes)
@@
 		(dnp no)
 		(property "Reference" "JP1"
-			(at 349.504 76.454 90)
+			(at 353.314 76.454 90)
 			(effects
 				(font
@@
 		)
 		(property "Value" "."
-			(at 353.568 81.788 90)
+			(at 357.378 81.788 90)
 			(effects
 				(font
@@
 		)
 		(property "Footprint" "Connector_PinHeader_2.54mm:PinHeader_1x03_P2.54mm_Vertical"
-			(at 355.6 80.01 0)
+			(at 359.41 80.01 0)
 			(effects
 				(font
@@
 		)
 		(property "Datasheet" "~"
-			(at 355.6 80.01 0)
+			(at 359.41 80.01 0)
 			(effects
 				(font
@@
 		)
 		(property "Description" "Jumper, 3-pole, both open"
-			(at 355.6 80.01 0)
+			(at 359.41 80.01 0)
 			(effects
 				(font
@@
 	(symbol
 		(lib_id "power:GND")
-		(at 355.6 86.36 0)
+		(at 359.41 86.36 0)
 		(unit 1)
 		(exclude_from_sim no)
@@
 		(dnp no)
 		(property "Reference" "#PWR073"
-			(at 355.6 92.71 0)
+			(at 359.41 92.71 0)
 			(effects
 				(font
@@
 		)
 		(property "Value" "GND"
-			(at 355.6 90.678 0)
+			(at 359.41 90.678 0)
 			(effects
 				(font
@@
 		)
 		(property "Footprint" ""
-			(at 355.6 86.36 0)
+			(at 359.41 86.36 0)
 			(effects
 				(font
@@
 		)
 		(property "Datasheet" ""
-			(at 355.6 86.36 0)
+			(at 359.41 86.36 0)
 			(effects
 				(font
@@
 		)
 		(property "Description" "Power symbol creates a global label with name \"GND\" , ground"
-			(at 355.6 86.36 0)
+			(at 359.41 86.36 0)
 			(effects
 				(font
@@
 			)
 		)
-		(property "Value" "74LS240"
+		(property "Value" "74HCT240"
 			(at 315.8333 20.32 0)
 			(effects
@@
 	)
 	(symbol
+		(lib_id "Connector_Generic:Conn_01x01")
+		(at 83.82 40.64 0)
+		(mirror x)
+		(unit 1)
+		(exclude_from_sim no)
+		(in_bom yes)
+		(on_board yes)
+		(dnp no)
+		(property "Reference" "J22"
+			(at 86.106 40.64 0)
+			(effects
+				(font
+					(size 1.27 1.27)
+				)
+				(justify left)
+			)
+		)
+		(property "Value" "Conn_01x01"
+			(at 86.36 39.3701 0)
+			(effects
+				(font
+					(size 1.27 1.27)
+				)
+				(justify left)
+				(hide yes)
+			)
+		)
+		(property "Footprint" "Connector_PinHeader_1.27mm:PinHeader_1x01_P1.27mm_Vertical"
+			(at 83.82 40.64 0)
+			(effects
+				(font
+					(size 1.27 1.27)
+				)
+				(hide yes)
+			)
+		)
+		(property "Datasheet" "~"
+			(at 83.82 40.64 0)
+			(effects
+				(font
+					(size 1.27 1.27)
+				)
+				(hide yes)
+			)
+		)
+		(property "Description" "Generic connector, single row, 01x01, script generated (kicad-library-utils/schlib/autogen/connector/)"
+			(at 83.82 40.64 0)
+			(effects
+				(font
+					(size 1.27 1.27)
+				)
+				(hide yes)
+			)
+		)
+		(pin "1"
+		)
+		(instances
+			(project "Exorset_Floppy"
+				(path "/05fb24d5-db99-47c3-b50e-9b588fa507ac/a1c0351e-a831-4754-8be5-6f4bd5bad354"
+					(reference "J22")
+					(unit 1)
+				)
+			)
+		)
+	)
+	(symbol
 		(lib_id "74xx:74LS74")
 		(at 191.77 97.79 0)
@@
 					(unit 1)
 				)
+			)
+		)
+	)
+	(symbol
+		(lib_id "Connector_Generic:Conn_01x01")
+		(at 346.71 76.2 0)
+		(mirror x)
+		(unit 1)
+		(exclude_from_sim no)
+		(in_bom yes)
+		(on_board yes)
+		(dnp no)
+		(property "Reference" "J21"
+			(at 348.996 76.2 0)
+			(effects
+				(font
+					(size 1.27 1.27)
+				)
+				(justify left)
+			)
+		)
+		(property "Value" "Conn_01x01"
+			(at 349.25 74.9301 0)
+			(effects
+				(font
+					(size 1.27 1.27)
+				)
+				(justify left)
+				(hide yes)
+			)
+		)
+		(property "Footprint" "Connector_PinHeader_1.27mm:PinHeader_1x01_P1.27mm_Vertical"
+			(at 346.71 76.2 0)
+			(effects
+				(font
+					(size 1.27 1.27)
+				)
+				(hide yes)
+			)
+		)
+		(property "Datasheet" "~"
+			(at 346.71 76.2 0)
+			(effects
+				(font
+					(size 1.27 1.27)
+				)
+				(hide yes)
+			)
+		)
+		(property "Description" "Generic connector, single row, 01x01, script generated (kicad-library-utils/schlib/autogen/connector/)"
+			(at 346.71 76.2 0)
+			(effects
+				(font
+					(size 1.27 1.27)
+				)
+				(hide yes)
+			)
+		)
+		(pin "1"
+		)
+		(instances
+			(project "Exorset_Floppy"
+				(path "/05fb24d5-db99-47c3-b50e-9b588fa507ac/a1c0351e-a831-4754-8be5-6f4bd5bad354"
+					(reference "J21")
+					(unit 1)
+				)

Commit message: first test with exordisk board, GALs new
Other:
- note added: "PROBLEM!"
- note added: "Problems (needs fixing in next Version): U23-2 needs to go to +5V, R4 from 47k -> 100k, C7 from 100u -> 220u U5-15 wrong, needs to go to U5-11 maybe more Testpoints - look in AN764"
Changed lines of the file:
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@@
 		)
 	)
+	(text "Problems (needs fixing in next Version):\nU23-2 needs to go to +5V,\nR4 from 47k -> 100k, C7 from 100u -> 220u\nU5-15 wrong, needs to go to U5-11\nmaybe more Testpoints - look in AN764"
+		(exclude_from_sim no)
+		(at 359.918 256.286 0)
+		(effects
+			(font
+				(size 1.27 1.27)
+			)
+			(justify left)
+		)
+	)
 	(text "D"
 		(exclude_from_sim no)
@@
 		)
 	)
+	(text "PROBLEM!"
+		(exclude_from_sim no)
+		(at 177.038 251.206 0)
+		(effects
+			(font
+				(size 1.27 1.27)
+				(thickness 0.254)
+				(bold yes)
+			)
+			(justify left)
+		)
+	)
 	(text "SM: Sync Match"
 		(exclude_from_sim no)
@@
 		)
 	)
+	(text "PROBLEM!"
+		(exclude_from_sim no)
+		(at 202.184 42.672 0)
+		(effects
+			(font
+				(size 1.27 1.27)
+				(thickness 0.254)
+				(bold yes)
+			)
+			(justify left)
+		)
+	)
 	(text "Jumper left of\nFloppy Connector"
 		(exclude_from_sim no)
@@
 		)
 	)
+	(polyline
+		(pts
+			(xy 171.45 252.73) (xy 176.53 252.095)
+		)
+		(stroke
+			(width 0)
+			(type default)
+		)
+	)
 	(wire
 		(pts
@@
 		)
 	)
+	(polyline
+		(pts
+			(xy 202.565 43.815) (xy 211.455 43.815)
+		)
+		(stroke
+			(width 0)
+			(type default)
+		)
+	)
 	(wire
 		(pts
@@
 		)
 	)
+	(polyline
+		(pts
+			(xy 211.455 43.815) (xy 218.44 41.91)
+		)
+		(stroke
+			(width 0)
+			(type default)
+		)
+	)
 	(wire
 		(pts
@@
 	(polyline
 		(pts
+			(xy 175.895 255.27) (xy 176.53 252.095)
+		)
+		(stroke
+			(width 0)
+			(type default)
+		)
+	)
+	(polyline
+		(pts
 			(xy 367.03 101.6) (xy 367.665 100.965)
 		)
@@
 		)
 		(stroke
+			(width 0)
+			(type default)
+		)
+	)
+	(polyline
+		(pts
+			(xy 186.69 252.095) (xy 176.53 252.095)
+		)
+		(stroke

Commit message: exordisk schematic updated, first working version
Parts:
- U24: value 74HC164 -> 74HCT164
Other:
- note added: "D0..3 are conn. to GND in AN764. Since there is no Load it doesn't matter."
- note added: "Data Recovery Circuit (see AN-764). Also read AN-535 (Phase-Locked Loop Design Fundamentals)."
- note added: "I used a 74HCT73 instead of the '76. Different Pinout though!"
- note added: "MC4044 aka MC4344."
- note added: "NMI Delay 0.8s Used for Timeout."
- note added: "OK, wrong in orig. schematics or different drive."
- note added: "PROBLEM Double Pin15 - RdCLK is Pin 5, Double Pin8,"
- note added: "Problems (needs fixing in next Version): U23-2 and U23-10 needs to go to +5V, R4 from 47k -> 100k, C7 from 100u -> 220u, U5-15 wrong, needs to go to U5-11, maybe more Testpoints - look in AN764, SEL2 and SEL3 should NOT be inverted, U34 has Datalines switched: D0->D7, D1->D6,..., U20 A0 and A1 are switched, U14 forgot +5V on Pin 14 and GND on Pin 7, U21-13 must conn. to GND (or maybe open?), MC85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"
- note added: "Reference Counter"
- note added: "Switch Clock Rate Latch"
- note added: "Testpoint missing! (C)"
- note added: "Testpoints missing! (En_CRC and not Q)"
- note added: "Testpoints missing! (Q0 and Q3)"
- note added: "Testpoints missing! (Sync Match and SM Latch Q and not Q)"
- note added: "U5, U28 and U29 are 74161 in the orig. Exordisk Controller. Diff. is only in the Reset. Since the Reset is not used the 74F163 is fine."
- note added: "Use U23A instead of U9! Tested the '123 and it works fine. Ditch the NE555!"
- note added: "Use a second '244 and a '04 for the input signals and as inverter for the MOT signal. Also: connect the HLD Signal."
- note added: "alternative for U13 (74LS91). Tested! Works fine."
- note added: "alternative for the MC4024 can be: 74LS624 or '324 74LS627 or '327 ( 'x27 is pincompatible)"
- note added: "div9"
- note removed: "0.8s"
- note removed: "Data Recovery Circuit (see AN-764)"
- note removed: "Problems (needs fixing in next Version): U23-2 needs to go to +5V, R4 from 47k -> 100k, C7 from 100u -> 220u U5-15 wrong, needs to go to U5-11 maybe more Testpoints - look in AN764"
- note removed: "Sw. Clock Rate Latch"
- note removed: "Use U23A instead of U9!"
- note removed: "alternative for U13 (74LS91)"
- moved on the sheet: JP2, JP6, U21B, U21C
