File: ExorsetFloppy/Exordisk_v1/Exordisk_v1.kicad_pcb (KiCad board)
At the start: 2 copper layers, 160 x 100 mm, 119 parts, among them J1 BUS, J10 Conn_01x01, J11 Conn_01x01, J12 Conn_01x01, J13 Conn_01x01, J14 Conn_01x01, J15 Conn_01x01, J16 Conn_01x01, J17 Conn_01x01, J18 Conn_01x01, J19 Conn_02x02_Odd_Even, J2 Floppy, J20 Conn_01x01, J21 Conn_01x01, J22 Conn_01x01, J23 Conn_01x01, J24 Conn_01x01, J25 Conn_01x01, J26 Conn_01x01, J27 Conn_01x01, J28 Conn_01x01, J29 Conn_01x01, J3 Conn_01x01, J30 Conn_01x01, J31 Conn_01x01, J32 Conn_01x01, J33 Conn_01x01, J34 Conn_01x01, J35 Conn_01x01, J36 Conn_01x01, J37 Conn_01x01, J38 Conn_01x01, J39 Conn_01x01, J4 Conn_01x01, J40 Conn_01x01, J41 Conn_01x01, J42 SS/DS, J5 Conn_01x01, J6 Conn_01x01, J7 Conn_01x17, J8 Conn_01x01, J9 Conn_01x01, Q1 BC337, U1 GAL22V10, U10 GAL16V8, U11 74HCT74, U12 74HCT74, U14 27C64, U15 74HCT04, U16 74HCT74, U17 74HCT00, U18 74HCT74, U19 74LS112, U2 74HCT74, U20 68B21, U21 MC4024, U22 74LS157, U23 74LS123, U24 74HCT164, U25 74LS04, U27 MC4044, U28 74F163, U29 74F163, U3 74HC245, U34 6852_DIL24, U4 MC8506_new, U5 74F163, U6 74LS139, U7 74HCT240, U8 74HCT244, U9 74LS32, Y1 1M

Commit message: exordisk firmware first working for DS
Parts:
- moved D6 0.52 mm to (184.8, 123.9), turned to 90 degrees
- moved U9 0.25 mm to (174.4, 135.5)
- moved D3 0.09 mm to (180.6, 131.7), turned to 0 degrees
- moved D5 0.09 mm to (189.4, 123.9), turned to 90 degrees
- moved D4 0.07 mm to (185.9, 131.7), turned to 180 degrees
Connections:
- D3 pad 1: /Floppy Logic/PA5 -> Net-(D3-K)
- D3 pad 2: Net-(D3-A) -> /Floppy Logic/PA5
- D4 pad 1: /Floppy Logic/PA5 -> Net-(D4-K)
- D4 pad 2: Net-(D4-A) -> /Floppy Logic/PA5
- D5 pad 1: /Floppy Logic/PA5 -> Net-(D5-K)
- D5 pad 2: Net-(D5-A) -> /Floppy Logic/PA5
- D6 pad 1: /Floppy Logic/PA5 -> Net-(D6-K)
- D6 pad 2: Net-(D6-A) -> /Floppy Logic/PA5
- U9 pad 11: Net-(D6-A) -> Net-(D6-K)
- U9 pad 3: Net-(D3-A) -> Net-(D3-K)
- U9 pad 6: Net-(D4-A) -> Net-(D4-K)
- U9 pad 8: Net-(D5-A) -> Net-(D5-K)
Routing:
- net /Floppy Logic/MOFF: track 33.3 -> 42.2 mm, vias 1 -> 2
- net Net-(U20-CA1): track 28.9 -> 34.3 mm
- net Net-(J26-Pin_1): track 82.4 -> 78.2 mm
- net Net-(D4-A): track 4.07 -> 0.00 mm
- net Net-(D3-K): track 0.00 -> 4.00 mm
- net Net-(D4-K): track 0.00 -> 3.97 mm
- net Net-(D3-A): track 3.82 -> 0.00 mm
- net Net-(D6-A): track 3.55 -> 0.00 mm
- net Net-(D6-K): track 0.00 -> 3.45 mm
- net Net-(D5-K): track 0.00 -> 2.63 mm
- net Net-(D5-A): track 2.45 -> 0.00 mm
- net /Floppy Logic/DS0: track 58.3 -> 56.6 mm
- net /Floppy Logic/TG43: track 21.0 -> 22.3 mm
- net /Floppy Logic/TXD: track 100.5 -> 99.4 mm
- net /Floppy Logic/DS3: track 65.1 -> 66.1 mm, vias 3 -> 2
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